File: TractorKit-Navis-Board.sch (KiCad schematic (older format))
At the start: 26 parts, among them J1 POWER, J2 GPS_I2C, J3 GPS_UART, J4 GPS_A, J5 GPS_B, U1 AMS1117-3.3, U2 ACS711xLCTR-12AB, U3 ESP32-WROOM-32

Commit message: Ready for panelization
Parts:
- D1: footprint (none) -> LED_SMD:LED_0603_1608Metric_Pad1.05x0.95mm_HandSolder
- J4: footprint (none) -> Connector_PinHeader_2.54mm:PinHeader_1x06_P2.54mm_Vertical
- J5: footprint (none) -> Connector_PinHeader_2.54mm:PinHeader_1x04_P2.54mm_Vertical
- R1, R2, R3: footprint Resistor_THT:R_Axial_DIN0207_L6.3mm_D2.5mm_P10.16mm_Horizontal -> Resistor_SMD:R_0603_1608Metric_Pad1.05x0.95mm_HandSolder
- R4: footprint (none) -> Resistor_SMD:R_0603_1608Metric_Pad1.05x0.95mm_HandSolder
- TP1, TP2, TP3, TP4, TP5: footprint TestPoint:TestPoint_Pad_D1.5mm -> TestPoint:TestPoint_Pad_D1.0mm
Connections:
- net AN_CURR: now also U3.9 (IO33)
- net AN_VOLT: now also U3.6 (IO34)
- no-connect marks 25 -> 23
Other:
- moved on the sheet: D1, R4
Changed lines of the file:
@@
 F 0 "TP5" V 2150 7150 50  0000 L CNN
 F 1 "SERVICE_GND" V 2150 7350 50  0000 L CNN
-F 2 "TestPoint:TestPoint_Pad_D1.5mm" H 2350 6950 50  0001 C CNN
+F 2 "TestPoint:TestPoint_Pad_D1.0mm" H 2350 6950 50  0001 C CNN
 F 3 "~" H 2350 6950 50  0001 C CNN
 	1    2150 6950
@@
 F 0 "TP3" V 2150 6950 50  0000 L CNN
 F 1 "SERVICE_RX" V 2150 7150 50  0000 L CNN
-F 2 "TestPoint:TestPoint_Pad_D1.5mm" H 2350 6750 50  0001 C CNN
+F 2 "TestPoint:TestPoint_Pad_D1.0mm" H 2350 6750 50  0001 C CNN
 F 3 "~" H 2350 6750 50  0001 C CNN
 	1    2150 6750
@@
 F 0 "TP2" V 2150 6850 50  0000 L CNN
 F 1 "SERVICE_TX" V 2150 7050 50  0000 L CNN
-F 2 "TestPoint:TestPoint_Pad_D1.5mm" H 2350 6650 50  0001 C CNN
+F 2 "TestPoint:TestPoint_Pad_D1.0mm" H 2350 6650 50  0001 C CNN
 F 3 "~" H 2350 6650 50  0001 C CNN
 	1    2150 6650
@@
 F 0 "TP1" V 2150 6750 50  0000 L CNN
 F 1 "SERVICE_BOOT" V 2150 6950 50  0000 L CNN
-F 2 "TestPoint:TestPoint_Pad_D1.5mm" H 2350 6550 50  0001 C CNN
+F 2 "TestPoint:TestPoint_Pad_D1.0mm" H 2350 6550 50  0001 C CNN
 F 3 "~" H 2350 6550 50  0001 C CNN
 	1    2150 6550
@@
 F 0 "TP4" V 2150 7050 50  0000 L CNN
 F 1 "SERVICE_3V3" V 2150 7250 50  0000 L CNN
-F 2 "TestPoint:TestPoint_Pad_D1.5mm" H 2350 6850 50  0001 C CNN
+F 2 "TestPoint:TestPoint_Pad_D1.0mm" H 2350 6850 50  0001 C CNN
 F 3 "~" H 2350 6850 50  0001 C CNN
 	1    2150 6850
@@
 F 0 "R1" V 2350 4900 50  0000 C CNN
 F 1 "10k" V 2250 4900 50  0000 C CNN
-F 2 "Resistor_THT:R_Axial_DIN0207_L6.3mm_D2.5mm_P10.16mm_Horizontal" V 2380 4900 50  0001 C CNN
+F 2 "Resistor_SMD:R_0603_1608Metric_Pad1.05x0.95mm_HandSolder" V 2380 4900 50  0001 C CNN
 F 3 "~" H 2450 4900 50  0001 C CNN
 	1    2450 4900
@@
 F 0 "R2" V 2850 4900 50  0000 C CNN
 F 1 "1k" V 2750 4900 50  0000 C CNN
-F 2 "Resistor_THT:R_Axial_DIN0207_L6.3mm_D2.5mm_P10.16mm_Horizontal" V 2880 4900 50  0001 C CNN
+F 2 "Resistor_SMD:R_0603_1608Metric_Pad1.05x0.95mm_HandSolder" V 2880 4900 50  0001 C CNN
 F 3 "~" H 2950 4900 50  0001 C CNN
 	1    2950 4900
@@
 Wire Wire Line
 	3200 4900 3100 4900
-Wire Wire Line
-	2300 3700 2300 3600
 Wire Wire Line
 	2300 3600 1100 3600
@@
 F 0 "R3" H 9500 3250 50  0000 C CNN
 F 1 "10k" H 9750 3250 50  0000 C CNN
-F 2 "Resistor_THT:R_Axial_DIN0207_L6.3mm_D2.5mm_P10.16mm_Horizontal" V 9530 3250 50  0001 C CNN
+F 2 "Resistor_SMD:R_0603_1608Metric_Pad1.05x0.95mm_HandSolder" V 9530 3250 50  0001 C CNN
 F 3 "~" H 9600 3250 50  0001 C CNN
 	1    9600 3250
@@
 F 0 "J4" H 6250 4250 50  0000 C CNN
 F 1 "GPS_A" H 6250 4350 50  0000 C CNN
-F 2 "" H 6050 4300 50  0001 C CNN
+F 2 "Connector_PinHeader_2.54mm:PinHeader_1x06_P2.54mm_Vertical" H 6050 4300 50  0001 C CNN
 F 3 "~" H 6050 4300 50  0001 C CNN
 	1    6050 4300
@@
 F 0 "J5" H 6250 4800 50  0000 C CNN
 F 1 "GPS_B" H 6250 4900 50  0000 C CNN
-F 2 "" H 6050 4850 50  0001 C CNN
+F 2 "Connector_PinHeader_2.54mm:PinHeader_1x04_P2.54mm_Vertical" H 6050 4850 50  0001 C CNN
 F 3 "~" H 6050 4850 50  0001 C CNN
 	1    6050 4850
@@
 NoConn ~ 7900 4900
 NoConn ~ 7900 5000
-NoConn ~ 7900 5100
-NoConn ~ 7900 5200
 NoConn ~ 7900 5300
 $Comp
@@
 L Device:R R4
 U 1 1 5F209256
-P 7450 4950
-F 0 "R4" H 7520 4996 50  0000 L CNN
-F 1 "R" H 7520 4905 50  0000 L CNN
-F 2 "" V 7380 4950 50  0001 C CNN
-F 3 "~" H 7450 4950 50  0001 C CNN
-	1    7450 4950
+P 6850 4950
+F 0 "R4" H 6920 4996 50  0000 L CNN
+F 1 "R" H 6920 4905 50  0000 L CNN
+F 2 "Resistor_SMD:R_0603_1608Metric_Pad1.05x0.95mm_HandSolder" V 6780 4950 50  0001 C CNN
+F 3 "~" H 6850 4950 50  0001 C CNN
+	1    6850 4950
 	1    0    0    -1
 $EndComp
@@
 L Device:LED D1
 U 1 1 5F209961
-P 7450 5350
-F 0 "D1" V 7489 5233 50  0000 R CNN
-F 1 "LED" V 7398 5233 50  0000 R CNN
-F 2 "" H 7450 5350 50  0001 C CNN
-F 3 "~" H 7450 5350 50  0001 C CNN
-	1    7450 5350
-	0    -1   -1   0
-$EndComp
-Wire Wire Line
-	7900 4700 7450 4700
-Wire Wire Line
-	7450 4700 7450 4800
-Wire Wire Line
-	7450 5200 7450 5100
+P 6850 5350
+F 0 "D1" V 6889 5233 50  0000 R CNN
+F 1 "LED" V 6798 5233 50  0000 R CNN
+F 2 "LED_SMD:LED_0603_1608Metric_Pad1.05x0.95mm_HandSolder" H 6850 5350 50  0001 C CNN
+F 3 "~" H 6850 5350 50  0001 C CNN
+	1    6850 5350
+	0    -1   -1   0
+$EndComp
+Wire Wire Line
+	7900 4700 6850 4700
+Wire Wire Line
+	6850 4700 6850 4800
+Wire Wire Line
+	6850 5200 6850 5100
 $Comp
 L power:GND #PWR024
 U 1 1 5F2174D8
-P 7450 5600
-F 0 "#PWR024" H 7450 5350 50  0001 C CNN
-F 1 "GND" H 7455 5427 50  0000 C CNN
-F 2 "" H 7450 5600 50  0001 C CNN
-F 3 "" H 7450 5600 50  0001 C CNN
-	1    7450 5600
-	1    0    0    -1
-$EndComp
-Wire Wire Line
-	7450 5600 7450 5500
+P 6850 5600
+F 0 "#PWR024" H 6850 5350 50  0001 C CNN
+F 1 "GND" H 6855 5427 50  0000 C CNN
+F 2 "" H 6850 5600 50  0001 C CNN
+F 3 "" H 6850 5600 50  0001 C CNN
+	1    6850 5600
+	1    0    0    -1
+$EndComp
+Wire Wire Line
+	6850 5600 6850 5500
+Wire Wire Line
+	2300 3600 2300 3700
+Text Label 7300 5100 0    50   ~ 0
+AN_CURR
+Text Label 7300 5200 0    50   ~ 0
+AN_VOLT
+Wire Wire Line
+	7900 5100 7300 5100
+Wire Wire Line
+	7300 5200 7900 5200
 Wire Bus Line
 	2600 6250 2600 6650
